Commit message: Implement move_base, navigation, slam

File: haruna/urdf/test.urdf (robot description, URDF)
Before this commit: robot test, 4 links, 3 joints
Links:
- added link laser
Joints:
- added joint body_to_laser: type fixed, parent body, child laser, origin xyz=0.22 0 0.18 rpy=0 3.14 0
- joint left_wheel_joint: origin xyz=0.0 0.17 0.0 rpy=0.0 0.0 0.0 -> xyz=0.0 0.17055 0.0 rpy=0.0 0.0 0.0
- joint right_wheel_joint: origin xyz=0.0 -0.17 0.0 rpy=0.0 0.0 3.14 -> xyz=0.0 -0.17055 0.0 rpy=0.0 0.0 3.14

Commit message: wip

File: haruna/urdf/test.urdf (robot description, URDF)
Before this commit: robot test, 4 links, 3 joints
Links:
- added link laser
Joints:
- added joint body_to_laser: type fixed, parent body, child laser, origin xyz=0.24 0 0 rpy=0 3.14 0
- joint left_wheel_joint: origin xyz=0.0 0.17 0.0 rpy=0.0 0.0 0.0 -> xyz=0.0 0.1721 0.0 rpy=0.0 0.0 0.0
- joint right_wheel_joint: origin xyz=0.0 -0.17 0.0 rpy=0.0 0.0 3.14 -> xyz=0.0 -0.1721 0.0 rpy=0.0 0.0 3.14

Commit message: aa

File: haruna/urdf/test.urdf (robot description, URDF)
Before this commit: robot test, 5 links, 4 joints
Joints:
- joint body_to_laser: origin xyz=0.24 0 0 rpy=0 3.14 0 -> xyz=0.22 0 0 rpy=0 3.14 0

Commit message: a

File: haruna/urdf/test.urdf (robot description, URDF)
Before this commit: robot test, 5 links, 4 joints
Joints:
- joint body_to_laser: origin xyz=0.22 0 0 rpy=0 3.14 0 -> xyz=0.22 0 0.18 rpy=0 3.14 0

Commit message: b

File: haruna/urdf/test.urdf (robot description, URDF)
Before this commit: robot test, 5 links, 4 joints
Joints:
- joint left_wheel_joint: origin xyz=0.0 0.1721 0.0 rpy=0.0 0.0 0.0 -> xyz=0.0 0.17055 0.0 rpy=0.0 0.0 0.0
- joint right_wheel_joint: origin xyz=0.0 -0.1721 0.0 rpy=0.0 0.0 3.14 -> xyz=0.0 -0.17055 0.0 rpy=0.0 0.0 3.14
