Commit message: add urdf and launch

File: haruna_gazebo/urdf/haruna.urdf.xacro (robot description, xacro)
@@ -1,71 +1,178 @@
-<?xml version="1.0"?>
-<robot name="haruna" xmlns:xacro="http://wiki.ros.org/xacro">
-    <xacro:property name="wheelwidth" value="0.085" />
-    <xacro:property name="wheellen" value="0.075" />
-    <xacro:property name="bodywidth" value="0.25" />
-    <xacro:property name="bodylen" value="0.01" />
-    <xacro:property name="pi" value="3.1415" />
-    <xacro:macro name="default_inertial" params="mass">
-        <inertial>
-            <mass value="${mass}" />
-            <inertia ixx="1.0" ixy="0.0" ixz="0.0" iyy="1.0" iyz="0.0" izz="1.0" />
-        </inertial>
-    </xacro:macro>
-    <link name="base_link" />
-    <joint name="base_to_body" type="fixed">
-        <origin xyz="0.0 0.0 0.12" rpy="0.0 0.0 0.0" />
-        <parent link="base_link"/>
-        <child link="body"/>
-    </joint>
-    <link name="body">
-        <visual>
-            <origin xyz="0.0 0.0 0.05" rpy="0.0 0.0 0.0"/>
-            <geometry>
-                <cylinder radius="${bodywidth}" length="${bodylen}" />
-            </geometry>
-            <material name="body">
-                <color rgba="0.8 0.8 0.8 0.5"/>
-            </material>
-        </visual>
-    </link>
-    <joint name="left_wheel_joint" type="continuous">
-	    <origin xyz="0.0 0.17055 0.0" rpy="0.0 0.0 0.0"/>
-	    <axis xyz="0 1 0"/>
-	    <parent link="body"/>
-	    <child link="left_wheel_link"/>
-    </joint>
-    <link name="left_wheel_link">
-        <visual>
-            <origin xyz="0.0 0.0 0.0" rpy="1.57 0.0 0.0"/>
-            <geometry>
-                <cylinder radius="${wheelwidth}" length="${wheellen}"/>
-            </geometry>
-            <material name="wheel">
-                <color rgba="0.8 0.8 0.8 1.0"/>
-            </material>
-        </visual>
-    </link>
-    <joint name="right_wheel_joint" type="continuous">
-        <origin xyz="0.0 -0.17055 0.0" rpy="0.0 0.0 ${pi}"/>
-        <axis xyz="0 1 0"/>
-        <parent link="body"/>
-        <child link="right_wheel_link"/>
-    </joint>
-    <link name="right_wheel_link">
-        <visual>
-            <origin xyz="0.0 0.0 0.0" rpy="${-pi/2} 0.0 0.0"/>
-            <geometry>
-                <cylinder radius="${wheelwidth}" length="${wheellen}"/>
-            </geometry>
-            <material name="wheel">
-                <color rgba="0.8 0.8 0.8 1.0"/>
-            </material>
-        </visual>
-    </link>
-    <link name="laser" />
-    <joint name="body_to_laser" type="fixed">
-        <parent link="body"/>
-        <child link="laser"/>
-        <origin rpy="0 3.14 0" xyz="0.22 0 0.18"/>
-    </joint>
+<?xml version="1.0" ?>
+<robot name="haruna" xmlns:xacro="http://www.ros.org/wiki/xacro">
+<!-- <xacro:include filename="$(find haruna_gazebo)/urdf/materials.xacro" /> -->
+<!-- <xacro:include filename="$(find haruna_gazebo)/urdf/haruna.trans" /> -->
+<!-- <xacro:include filename="$(find haruna_gazebo)/urdf/haruna.gazebo" /> -->
+<link name="base_link">
+  <!-- <inertial>
+    <origin xyz="1.0338131004861055e-16 5.1690655024305274e-17 0.157" rpy="0 0 0"/>
+    <mass value="1.381203895667492"/>
+    <inertia ixx="0.019888" iyy="0.023891" izz="0.043779" ixy="0.0" iyz="0.0" ixz="0.0"/>
+  </inertial> -->
+  <visual>
+    <origin xyz="0 0 0" rpy="0 0 0"/>
+    <geometry>
+      <mesh filename="../meshes/base_link.stl" scale="0.001 0.001 0.001"/>
+    </geometry>
+    <!-- <material name="silver"/> -->
+  </visual>
+  <collision>
+    <origin xyz="0 0 0" rpy="0 0 0"/>
+    <geometry>
+      <mesh filename="../meshes/base_link.stl" scale="0.001 0.001 0.001"/>
+    </geometry>
+  </collision>
+</link>
+<link name="front_leg_link_1">
+  <!-- <inertial>
+    <origin xyz="0.20000000000000004 0.0 -0.23149999999999998" rpy="0 0 0"/>
+    <mass value="0.11774999999999997"/>
+    <inertia ixx="0.000222" iyy="0.000222" izz="2e-06" ixy="0.0" iyz="0.0" ixz="0.0"/>
+  </inertial> -->
+  <visual>
+    <origin xyz="-0.0 -0.0 -0.313" rpy="0 0 0"/>
+    <geometry>
+      <mesh filename="../meshes/front_leg_link_1.stl" scale="0.001 0.001 0.001"/>
+    </geometry>
+    <!-- <material name="silver"/> -->
+  </visual>
+  <collision>
+    <origin xyz="-0.0 -0.0 -0.313" rpy="0 0 0"/>
+    <geometry>
+      <mesh filename="../meshes/front_leg_link_1.stl" scale="0.001 0.001 0.001"/>
+    </geometry>
+  </collision>
+</link>
+<link name="back_leg_link_1">
+  <!-- <inertial>
+    <origin xyz="-0.2 0.0 -0.23149999999999998" rpy="0 0 0"/>
+    <mass value="0.11775"/>
+    <inertia ixx="0.000222" iyy="0.000222" izz="2e-06" ixy="0.0" iyz="0.0" ixz="-0.0"/>
+  </inertial> -->
+  <visual>
+    <origin xyz="-0.0 -0.0 -0.313" rpy="0 0 0"/>
+    <geometry>
+      <mesh filename="../meshes/back_leg_link_1.stl" scale="0.001 0.001 0.001"/>
+    </geometry>
+    <!-- <material name="silver"/> -->
+  </visual>
+  <collision>
+    <origin xyz="-0.0 -0.0 -0.313" rpy="0 0 0"/>
+    <geometry>
+      <mesh filename="../meshes/back_leg_link_1.stl" scale="0.001 0.001 0.001"/>
+    </geometry>
+  </collision>
+</link>
+<link name="right_leg_link_1">
+  <!-- <inertial>
+    <origin xyz="0.0 -0.10865606936416185 -0.19859393063583816" rpy="0 0 0"/>
+    <mass value="0.06790249999999999"/>
+    <inertia ixx="3.8e-05" iyy="3.8e-05" izz="2e-06" ixy="-0.0" iyz="-2e-06" ixz="0.0"/>
+  </inertial> -->
+  <visual>
+    <origin xyz="-0.0 -0.0 -0.313" rpy="0 0 0"/>
+    <geometry>
+      <mesh filename="../meshes/right_leg_link_1.stl" scale="0.001 0.001 0.001"/>
+    </geometry>
+    <!-- <material name="silver"/> -->
+  </visual>
+  <collision>
+    <origin xyz="-0.0 -0.0 -0.313" rpy="0 0 0"/>
+    <geometry>
+      <mesh filename="../meshes/right_leg_link_1.stl" scale="0.001 0.001 0.001"/>
+    </geometry>
+  </collision>
+</link>
+<link name="left_leg_link_1">
+  <!-- <inertial>
+    <origin xyz="0.0 0.10865606936416185 -0.19859393063583816" rpy="0 0 0"/>
+    <mass value="0.06790249999999999"/>
+    <inertia ixx="3.8e-05" iyy="3.8e-05" izz="2e-06" ixy="0.0" iyz="2e-06" ixz="0.0"/>
+  </inertial> -->
+  <visual>
+    <origin xyz="-0.0 -0.0 -0.313" rpy="0 0 0"/>
+    <geometry>
+      <mesh filename="../meshes/left_leg_link_1.stl" scale="0.001 0.001 0.001"/>
+    </geometry>
+    <!-- <material name="silver"/> -->
+  </visual>
+  <collision>
+    <origin xyz="-0.0 -0.0 -0.313" rpy="0 0 0"/>
+    <geometry>
+      <mesh filename="../meshes/left_leg_link_1.stl" scale="0.001 0.001 0.001"/>
+    </geometry>
+  </collision>
+</link>
+<link name="left_wheel_link_1">
+  <!-- <inertial>
+    <origin xyz="-1.0685163737249417e-17 0.037500000000000006 0.0" rpy="0 0 0"/>
+    <mass value="13.363451575437157"/>
+    <inertia ixx="0.030402" iyy="0.048275" izz="0.030402" ixy="-0.0" iyz="0.0" ixz="-0.0"/>
+  </inertial> -->
+  <visual>
+    <origin xyz="-0.0 -0.1225 -0.085" rpy="0 0 0"/>
+    <geometry>
+      <mesh filename="../meshes/left_wheel_link_1.stl" scale="0.001 0.001 0.001"/>
+    </geometry>
+    <!-- <material name="silver"/> -->
+  </visual>
+  <collision>
+    <origin xyz="-0.0 -0.1225 -0.085" rpy="0 0 0"/>
+    <geometry>
+      <mesh filename="../meshes/left_wheel_link_1.stl" scale="0.001 0.001 0.001"/>
+    </geometry>
+  </collision>
+</link>
+<link name="right_wheel_link_1">
+  <!-- <inertial>
+    <origin xyz="-1.0685163737249417e-17 -0.037500000000000006 0.0" rpy="0 0 0"/>
+    <mass value="13.363451575437157"/>
+    <inertia ixx="0.030402" iyy="0.048275" izz="0.030402" ixy="-0.0" iyz="-0.0" ixz="-0.0"/>
+  </inertial> -->
+  <visual>
+    <origin xyz="-0.0 0.1225 -0.085" rpy="0 0 0"/>
+    <geometry>
+      <mesh filename="../meshes/right_wheel_link_1.stl" scale="0.001 0.001 0.001"/>
+    </geometry>
+    <!-- <material name="silver"/> -->
+  </visual>
+  <collision>
+    <origin xyz="-0.0 0.1225 -0.085" rpy="0 0 0"/>
+    <geometry>
+      <mesh filename="../meshes/right_wheel_link_1.stl" scale="0.001 0.001 0.001"/>
+    </geometry>
+  </collision>
+</link>
+<joint name="base_to_front_leg_joint" type="fixed">
+  <origin xyz="0.0 0.0 0.313" rpy="0 0 0"/>
+  <parent link="base_link"/>
+  <child link="front_leg_link_1"/>
+</joint>
+<joint name="base_to_back_leg_joint" type="fixed">
+  <origin xyz="0.0 0.0 0.313" rpy="0 0 0"/>
+  <parent link="base_link"/>
+  <child link="back_leg_link_1"/>
+</joint>
+<joint name="base_to_right_leg_joint" type="fixed">
+  <origin xyz="0.0 0.0 0.313" rpy="0 0 0"/>
+  <parent link="base_link"/>
+  <child link="right_leg_link_1"/>
+</joint>
+<joint name="base_to_left_leg_joint" type="fixed">
+  <origin xyz="0.0 0.0 0.313" rpy="0 0 0"/>
+  <parent link="base_link"/>
+  <child link="left_leg_link_1"/>
+</joint>
+<joint name="left_leg_to_left_wheel_joint" type="continuous">
+  <origin xyz="0.0 0.1225 -0.228" rpy="0 0 0"/>
+  <parent link="left_leg_link_1"/>
+  <child link="left_wheel_link_1"/>
+  <axis xyz="0.0 1.0 0.0"/>
+</joint>
+<joint name="right_leg_to_right_wheel_joint" type="continuous">
+  <origin xyz="0.0 -0.1225 -0.228" rpy="0 0 0"/>
+  <parent link="right_leg_link_1"/>
+  <child link="right_wheel_link_1"/>
+  <axis xyz="0.0 -1.0 0.0"/>
+</joint>
 </robot>

Commit message: update

File: haruna_gazebo/urdf/haruna.urdf.xacro (robot description, xacro)
@@ -2,6 +2,6 @@
 <robot name="haruna" xmlns:xacro="http://www.ros.org/wiki/xacro">
 <!-- <xacro:include filename="$(find haruna_gazebo)/urdf/materials.xacro" /> -->
-<!-- <xacro:include filename="$(find haruna_gazebo)/urdf/haruna.trans" /> -->
-<!-- <xacro:include filename="$(find haruna_gazebo)/urdf/haruna.gazebo" /> -->
+<xacro:include filename="$(find haruna_gazebo)/urdf/haruna.trans" />
+<xacro:include filename="$(find haruna_gazebo)/urdf/haruna.gazebo" />
 <link name="base_link">
   <!-- <inertial>
@@ -13,5 +13,5 @@
     <origin xyz="0 0 0" rpy="0 0 0"/>
     <geometry>
-      <mesh filename="../meshes/base_link.stl" scale="0.001 0.001 0.001"/>
+      <mesh filename="package://haruna_gazebo/meshes/base_link.stl" scale="0.001 0.001 0.001"/>
     </geometry>
     <!-- <material name="silver"/> -->
@@ -20,5 +20,5 @@
     <origin xyz="0 0 0" rpy="0 0 0"/>
     <geometry>
-      <mesh filename="../meshes/base_link.stl" scale="0.001 0.001 0.001"/>
+      <mesh filename="package://haruna_gazebo/meshes/base_link.stl" scale="0.001 0.001 0.001"/>
     </geometry>
   </collision>
@@ -33,5 +33,5 @@
     <origin xyz="-0.0 -0.0 -0.313" rpy="0 0 0"/>
     <geometry>
-      <mesh filename="../meshes/front_leg_link_1.stl" scale="0.001 0.001 0.001"/>
+      <mesh filename="package://haruna_gazebo/meshes/front_leg_link_1.stl" scale="0.001 0.001 0.001"/>
     </geometry>
     <!-- <material name="silver"/> -->
@@ -40,5 +40,5 @@
     <origin xyz="-0.0 -0.0 -0.313" rpy="0 0 0"/>
     <geometry>
-      <mesh filename="../meshes/front_leg_link_1.stl" scale="0.001 0.001 0.001"/>
+      <mesh filename="package://haruna_gazebo/meshes/front_leg_link_1.stl" scale="0.001 0.001 0.001"/>
     </geometry>
   </collision>
@@ -53,5 +53,5 @@
     <origin xyz="-0.0 -0.0 -0.313" rpy="0 0 0"/>
     <geometry>
-      <mesh filename="../meshes/back_leg_link_1.stl" scale="0.001 0.001 0.001"/>
+      <mesh filename="package://haruna_gazebo/meshes/back_leg_link_1.stl" scale="0.001 0.001 0.001"/>
     </geometry>
     <!-- <material name="silver"/> -->
@@ -60,5 +60,5 @@
     <origin xyz="-0.0 -0.0 -0.313" rpy="0 0 0"/>
     <geometry>
-      <mesh filename="../meshes/back_leg_link_1.stl" scale="0.001 0.001 0.001"/>
+      <mesh filename="package://haruna_gazebo/meshes/back_leg_link_1.stl" scale="0.001 0.001 0.001"/>
     </geometry>
   </collision>
@@ -73,5 +73,5 @@
     <origin xyz="-0.0 -0.0 -0.313" rpy="0 0 0"/>
     <geometry>
-      <mesh filename="../meshes/right_leg_link_1.stl" scale="0.001 0.001 0.001"/>
+      <mesh filename="package://haruna_gazebo/meshes/right_leg_link_1.stl" scale="0.001 0.001 0.001"/>
     </geometry>
     <!-- <material name="silver"/> -->
@@ -80,5 +80,5 @@
     <origin xyz="-0.0 -0.0 -0.313" rpy="0 0 0"/>
     <geometry>
-      <mesh filename="../meshes/right_leg_link_1.stl" scale="0.001 0.001 0.001"/>
+      <mesh filename="package://haruna_gazebo/meshes/right_leg_link_1.stl" scale="0.001 0.001 0.001"/>
     </geometry>
   </collision>
@@ -93,5 +93,5 @@
     <origin xyz="-0.0 -0.0 -0.313" rpy="0 0 0"/>
     <geometry>
-      <mesh filename="../meshes/left_leg_link_1.stl" scale="0.001 0.001 0.001"/>
+      <mesh filename="package://haruna_gazebo/meshes/left_leg_link_1.stl" scale="0.001 0.001 0.001"/>
     </geometry>
     <!-- <material name="silver"/> -->
@@ -100,5 +100,5 @@
     <origin xyz="-0.0 -0.0 -0.313" rpy="0 0 0"/>
     <geometry>
-      <mesh filename="../meshes/left_leg_link_1.stl" scale="0.001 0.001 0.001"/>
+      <mesh filename="package://haruna_gazebo/meshes/left_leg_link_1.stl" scale="0.001 0.001 0.001"/>
     </geometry>
   </collision>
@@ -113,5 +113,5 @@
     <origin xyz="-0.0 -0.1225 -0.085" rpy="0 0 0"/>
     <geometry>
-      <mesh filename="../meshes/left_wheel_link_1.stl" scale="0.001 0.001 0.001"/>
+      <mesh filename="package://haruna_gazebo/meshes/left_wheel_link_1.stl" scale="0.001 0.001 0.001"/>
     </geometry>
     <!-- <material name="silver"/> -->
@@ -120,5 +120,5 @@
     <origin xyz="-0.0 -0.1225 -0.085" rpy="0 0 0"/>
     <geometry>
-      <mesh filename="../meshes/left_wheel_link_1.stl" scale="0.001 0.001 0.001"/>
+      <mesh filename="package://haruna_gazebo/meshes/left_wheel_link_1.stl" scale="0.001 0.001 0.001"/>
     </geometry>
   </collision>
@@ -133,5 +133,5 @@
     <origin xyz="-0.0 0.1225 -0.085" rpy="0 0 0"/>
     <geometry>
-      <mesh filename="../meshes/right_wheel_link_1.stl" scale="0.001 0.001 0.001"/>
+      <mesh filename="package://haruna_gazebo/meshes/right_wheel_link_1.stl" scale="0.001 0.001 0.001"/>
     </geometry>
     <!-- <material name="silver"/> -->
@@ -140,5 +140,5 @@
     <origin xyz="-0.0 0.1225 -0.085" rpy="0 0 0"/>
     <geometry>
-      <mesh filename="../meshes/right_wheel_link_1.stl" scale="0.001 0.001 0.001"/>
+      <mesh filename="package://haruna_gazebo/meshes/right_wheel_link_1.stl" scale="0.001 0.001 0.001"/>
     </geometry>
   </collision>
