Commit message: update

File: haruna_gazebo/urdf/haruna.urdf (robot description, URDF)
Before this commit: robot haruna, 7 links, 6 joints
Links:
- added link laser_link, mass 1e-5; collision cylinder length=0.03 radius=0.015; visual cylinder length=0.03 radius=0.015
Joints:
- added joint base_to_laser: type fixed, parent base_link, child laser_link, origin xyz=0.2 0.0 0.17 rpy=0.0 0.0 0.0
