Commit message: add haruna_description and haruna_simulations

File: haruna_description/urdf/haruna.urdf (robot description, URDF)
Before this commit: robot haruna, 8 links, 7 joints
Links:
- removed link laser_link
- added link laser, mass 1e-5; collision cylinder length=0.03 radius=0.015; visual cylinder length=0.03 radius=0.015
- link back_leg_link_1: geometry collision mesh filename=package://haruna_description/meshes/back_leg_link_1.stl scale=0.001 0.001 0.001; visual mesh filename=package://haruna_description/meshes/back_leg_link_1.stl scale=0.001 0.001 0.001
- link base_link: geometry collision mesh filename=package://haruna_description/meshes/base_link.stl scale=0.001 0.001 0.001; visual mesh filename=package://haruna_description/meshes/base_link.stl scale=0.001 0.001 0.001
- link front_leg_link_1: geometry collision mesh filename=package://haruna_description/meshes/front_leg_link_1.stl scale=0.001 0.001 0.001; visual mesh filename=package://haruna_description/meshes/front_leg_link_1.stl scale=0.001 0.001 0.001
- link left_leg_link_1: geometry collision mesh filename=package://haruna_description/meshes/left_leg_link_1.stl scale=0.001 0.001 0.001; visual mesh filename=package://haruna_description/meshes/left_leg_link_1.stl scale=0.001 0.001 0.001
- link left_wheel_link_1: geometry collision mesh filename=package://haruna_description/meshes/left_wheel_link_1.stl scale=0.001 0.001 0.001; visual mesh filename=package://haruna_description/meshes/left_wheel_link_1.stl scale=0.001 0.001 0.001
- link right_leg_link_1: geometry collision mesh filename=package://haruna_description/meshes/right_leg_link_1.stl scale=0.001 0.001 0.001; visual mesh filename=package://haruna_description/meshes/right_leg_link_1.stl scale=0.001 0.001 0.001
- link right_wheel_link_1: geometry collision mesh filename=package://haruna_description/meshes/right_wheel_link_1.stl scale=0.001 0.001 0.001; visual mesh filename=package://haruna_description/meshes/right_wheel_link_1.stl scale=0.001 0.001 0.001
Joints:
- joint base_to_laser: child laser_link -> laser; origin xyz=0.2 0.0 0.17 rpy=0.0 0.0 0.0 -> xyz=0.2 0.0 0.17 rpy=0.0 3.14 0.0
